File: board/board.kicad_pcb (KiCad board)
At the start: 2 copper layers, 21 x 13 mm, 1 part

Commit message: initial
Parts:
- added J1: 018_QSPI, on_edge:on_edge_2x05_host, F.Cu at (140.0, 96.5)
- added J2: Micro_SD_Card_Det, Connector_Card:microSD_HC_Molex_104031-0811, F.Cu at (152.8, 96.5)
- LOGO1: moved to B.Cu
- moved LOGO1 3.00 mm to (152.8, 97.8), turned to 180 degrees
Routing:
- net GND: track 0.00 -> 37.5 mm, vias 0 -> 31
- net /sd/CS: track 0.00 -> 18.5 mm, vias 0 -> 1
- net /sd/SD1: track 0.00 -> 17.7 mm, vias 0 -> 2
- net /sd/3.3V: track 0.00 -> 16.8 mm, vias 0 -> 1
- net /sd/SD3: track 0.00 -> 16.7 mm, vias 0 -> 2
- net /sd/SD2: track 0.00 -> 16.6 mm
- net /sd/SD0: track 0.00 -> 16.5 mm
- net /sd/SCLK: track 0.00 -> 16.2 mm, vias 0 -> 1
- net /sd/SW1: track 0.00 -> 10.3 mm, vias 0 -> 1
- net /sd/SW0: track 0.00 -> 10.1 mm, vias 0 -> 1
- added copper zone on B.Cu, net GND
- added copper zone on F.Cu, net GND
Other:
- outline, holes or cut-outs redrawn
- board text added: "osf.018"
- board text added: "osf.b123.v1.0"
